Commit message: 작동 확인

File: config/turtlebot3_arm.ros2_control.xacro (robot description, xacro)
@@ -1,9 +1,9 @@
 <?xml version="1.0"?>
 <robot xmlns:xacro="http://www.ros.org/wiki/xacro">
-    <xacro:macro name="conveyor_belt_ros2_control" params="name">
+    <xacro:macro name="turtlebot3_arm_ros2_control" params="name">
         <ros2_control name="${name}" type="system">
           <hardware>
             <plugin>dynamixel_hardware_interface/DynamixelHardware</plugin>
-            <param name="port_name">/dev/ttyACM0</param>
+            <param name="port_name">/dev/ttyACM1</param>
             <param name="baud_rate">1000000</param>
             <param name="dynamixel_model_folder">/param/dxl_model</param>
@@ -30,5 +30,5 @@
           <gpio name="dxl1">
             <param name="type">dxl</param>
-            <param name="ID">3</param>
+            <param name="ID">19</param>
             <command_interface name="Goal Position"/>
             <state_interface name="Present Position"/>

File: config/turtlebot3_arm.urdf.xacro (robot description, xacro)
@@ -1,13 +1,13 @@
 <?xml version="1.0"?>
-<robot xmlns:xacro="http://www.ros.org/wiki/xacro" name="conveyor_belt">
+<robot xmlns:xacro="http://www.ros.org/wiki/xacro" name="turtlebot3_arm">
     <xacro:arg name="tf_prefix" default="" />
     <!-- Import control_xacro -->
-    <xacro:include filename="conveyor_belt.ros2_control.xacro" />
-    <xacro:conveyor_belt_ros2_control name="conveyor_belt"/>
+    <xacro:include filename="turtlebot3_arm.ros2_control.xacro" />
+    <xacro:turtlebot3_arm_ros2_control name="turtlebot3_arm"/>
     <link name="$(arg tf_prefix)base_link"/>
-    <link name="$(arg tf_prefix)conveyor_belt"/>
+    <link name="$(arg tf_prefix)turtlebot3_arm"/>
     <joint name="$(arg tf_prefix)joint1" type="revolute">
         <parent link="$(arg tf_prefix)base_link"/>
-        <child link="$(arg tf_prefix)conveyor_belt"/>
+        <child link="$(arg tf_prefix)turtlebot3_arm"/>
         <origin xyz="0 0 0" rpy="0 0 0"/>
         <axis xyz="1 0 0" />
